Commit message: update uav's model

File: src/ugv_description/urdf/ugv_shared.xacro (robot description, xacro)
@@ -94,4 +94,5 @@
     <xacro:property name="base_link_name" value="${robot_prefix}base_link" />
     <xacro:property name="computer_link" value="${robot_prefix}computer" />
+    <xacro:property name="tag16h5_plane_link" value="${robot_prefix}tag16h5_plane" />
     <xacro:property name="laser_link" value="${robot_prefix}laser" />
     <xacro:property name="imu_link_name" value="${robot_prefix}imu_link" />
@@ -186,4 +187,28 @@
       <xacro:box_inertial m="0.5" x="0.13" y="0.13" z="0.05" />
     </link>
+    <joint name="${robot_prefix}tag16h5_plane_joint" type="fixed">
+      <origin xyz="-0.15 0 0.1" rpy="0 0 0" />
+      <parent link="${computer_link}" />
+      <child link="${tag16h5_plane_link}" />
+    </joint>
+    <link name="${tag16h5_plane_link}">
+      <visual name="${robot_prefix}tag16h5_plane_body_visual">
+        <geometry>
+          <mesh filename="package://ugv_description/meshes/plane.dae" scale="1 1 1" />
+        </geometry>
+      </visual>
+      <visual name="${robot_prefix}tag16h5_plane_marker_visual">
+        <origin xyz="0 0 0.027" rpy="0 0 0" />
+        <geometry>
+          <mesh filename="package://ugv_description/meshes/tag16h5_plane.dae" scale="1 1 1" />
+        </geometry>
+      </visual>
+      <collision name="${robot_prefix}tag16h5_plane_collision">
+        <geometry>
+          <mesh filename="package://ugv_description/meshes/plane.dae" scale="1 1 1" />
+        </geometry>
+      </collision>
+      <xacro:box_inertial m="0.05" x="0.4" y="0.2" z="0.05" />
+    </link>
     <joint name="${robot_prefix}lidar_joint" type="fixed">
       <origin xyz="0.1 0 0.11" rpy="0 0 0" />

Commit message: refine vl

File: src/ugv_description/urdf/ugv_shared.xacro (robot description, xacro)
@@ -199,5 +199,5 @@
       </visual>
       <visual name="${robot_prefix}tag16h5_plane_marker_visual">
-        <origin xyz="0 0 0.027" rpy="0 0 0" />
+        <origin xyz="0.05 0 0.027" rpy="0 0 ${PI/2}" />
         <geometry>
           <mesh filename="package://ugv_description/meshes/tag16h5_plane.dae" scale="1 1 1" />

Commit message: refactor fusion

File: src/ugv_description/urdf/ugv_shared.xacro (robot description, xacro)
@@ -199,5 +199,5 @@
       </visual>
       <visual name="${robot_prefix}tag16h5_plane_marker_visual">
-        <origin xyz="0.05 0 0.027" rpy="0 0 ${PI/2}" />
+        <origin xyz="0.07 0 0.027" rpy="0 0 ${PI/2}" />
         <geometry>
           <mesh filename="package://ugv_description/meshes/tag16h5_plane.dae" scale="1 1 1" />

Commit message: refine sth

File: src/ugv_description/urdf/ugv_shared.xacro (robot description, xacro)
@@ -199,5 +199,5 @@
       </visual>
       <visual name="${robot_prefix}tag16h5_plane_marker_visual">
-        <origin xyz="0.07 0 0.027" rpy="0 0 ${PI/2}" />
+        <origin xyz="0.07 0 0.027" rpy="0 0 -${PI/2}" />
         <geometry>
           <mesh filename="package://ugv_description/meshes/tag16h5_plane.dae" scale="1 1 1" />

Commit message: refine nav2

File: src/ugv_description/urdf/ugv_shared.xacro (robot description, xacro)
@@ -212,5 +212,5 @@
     </link>
     <joint name="${robot_prefix}lidar_joint" type="fixed">
-      <origin xyz="0.1 0 0.11" rpy="0 0 0" />
+      <origin xyz="0.085 0 0.11" rpy="0 0 0" />
       <parent link="${base_link_name}" />
       <child link="${laser_link}" />

Commit message: refine nav2

File: src/ugv_description/urdf/ugv_shared.xacro (robot description, xacro)
@@ -94,5 +94,5 @@
     <xacro:property name="base_link_name" value="${robot_prefix}base_link" />
     <xacro:property name="computer_link" value="${robot_prefix}computer" />
-    <xacro:property name="tag16h5_plane_link" value="${robot_prefix}tag16h5_plane" />
+    <xacro:property name="tag36h11_plane_link" value="${robot_prefix}tag36h11_plane" />
     <xacro:property name="laser_link" value="${robot_prefix}laser" />
     <xacro:property name="imu_link_name" value="${robot_prefix}imu_link" />
@@ -187,22 +187,22 @@
       <xacro:box_inertial m="0.5" x="0.13" y="0.13" z="0.05" />
     </link>
-    <joint name="${robot_prefix}tag16h5_plane_joint" type="fixed">
+    <joint name="${robot_prefix}tag36h11_plane_joint" type="fixed">
       <origin xyz="-0.15 0 0.1" rpy="0 0 0" />
       <parent link="${computer_link}" />
-      <child link="${tag16h5_plane_link}" />
-    </joint>
-    <link name="${tag16h5_plane_link}">
-      <visual name="${robot_prefix}tag16h5_plane_body_visual">
+      <child link="${tag36h11_plane_link}" />
+    </joint>
+    <link name="${tag36h11_plane_link}">
+      <visual name="${robot_prefix}tag36h11_plane_body_visual">
         <geometry>
           <mesh filename="package://ugv_description/meshes/plane.dae" scale="1 1 1" />
         </geometry>
       </visual>
-      <visual name="${robot_prefix}tag16h5_plane_marker_visual">
-        <origin xyz="0.07 0 0.027" rpy="0 0 -${PI/2}" />
-        <geometry>
-          <mesh filename="package://ugv_description/meshes/tag16h5_plane.dae" scale="1 1 1" />
-        </geometry>
-      </visual>
-      <collision name="${robot_prefix}tag16h5_plane_collision">
+      <visual name="${robot_prefix}tag36h11_plane_marker_visual">
+        <origin xyz="0.03 0 0.027" rpy="0 0 0" />
+        <geometry>
+          <mesh filename="package://ugv_description/meshes/tag36h11_plane.dae" scale="1 1 1" />
+        </geometry>
+      </visual>
+      <collision name="${robot_prefix}tag36h11_plane_collision">
         <geometry>
           <mesh filename="package://ugv_description/meshes/plane.dae" scale="1 1 1" />

Commit message: refine nav2

File: src/ugv_description/urdf/ugv_shared.xacro (robot description, xacro)
@@ -199,5 +199,5 @@
       </visual>
       <visual name="${robot_prefix}tag36h11_plane_marker_visual">
-        <origin xyz="0.03 0 0.027" rpy="0 0 0" />
+        <origin xyz="0.03 0 0.027" rpy="0 0 ${PI/2}" />
         <geometry>
           <mesh filename="package://ugv_description/meshes/tag36h11_plane.dae" scale="1 1 1" />
